Commit message: Added moveit package for s650

File: adept_s650_support/urdf/s650_macro.xacro (robot description, xacro)
@@ -9,6 +9,6 @@
           <mesh filename="package://adept_s650_support/meshes/s650/visual/base_link.stl"/>
         </geometry>
-        <material name="White">
-          <color rgba="255 255 255 1.0"/>
+        <material name="Grey">
+          <color rgba="128 128 128 1.0"/>
         </material>
       </visual>
@@ -29,6 +29,6 @@
           <mesh filename="package://adept_s650_support/meshes/s650/visual/link_1.stl"/>
         </geometry>
-        <material name="White">
-          <color rgba="255 255 255 1.0"/>
+        <material name="Grey">
+          <color rgba="128 128 128 1.0"/>
         </material>
       </visual>
@@ -49,6 +49,6 @@
           <mesh filename="package://adept_s650_support/meshes/s650/visual/link_2.stl"/>
         </geometry>
-        <material name="White">
-          <color rgba="255 255 255 1.0"/>
+        <material name="Grey">
+          <color rgba="128 128 128 1.0"/>
         </material>
       </visual>
@@ -69,6 +69,6 @@
           <mesh filename="package://adept_s650_support/meshes/s650/visual/link_3.stl"/>
         </geometry>
-        <material name="White">
-          <color rgba="255 255 255 1.0"/>
+        <material name="Grey">
+          <color rgba="128 128 128 1.0"/>
         </material>
       </visual>
@@ -89,6 +89,6 @@
           <mesh filename="package://adept_s650_support/meshes/s650/visual/link_4.stl"/>
         </geometry>
-        <material name="White">
-          <color rgba="255 255 255 1.0"/>
+        <material name="Grey">
+          <color rgba="128 128 128 1.0"/>
         </material>
       </visual>
@@ -109,6 +109,6 @@
           <mesh filename="package://adept_s650_support/meshes/s650/visual/link_5.stl"/>
         </geometry>
-        <material name="White">
-          <color rgba="255 255 255 1.0"/>
+        <material name="Grey">
+          <color rgba="128 128 128 1.0"/>
         </material>
       </visual>

Commit message: Added robot_state node to driver

File: adept_s650_support/urdf/s650_macro.xacro (robot description, xacro)
@@ -1,3 +1,3 @@
-<?xml version="1.0" ?>
+<?xml version="1" ?>
 <robot xmlns:xacro="http://ros.org/wiki/xacro">
   <xacro:macro name="adept_s650" params="prefix">
@@ -9,6 +9,6 @@
           <mesh filename="package://adept_s650_support/meshes/s650/visual/base_link.stl"/>
         </geometry>
-        <material name="Grey">
-          <color rgba="128 128 128 1.0"/>
+        <material name="adept_grey">
+          <color rgba="0.5 0.5 0.5 1"/>
         </material>
       </visual>
@@ -18,6 +18,6 @@
           <mesh filename="package://adept_s650_support/meshes/s650/collision/base_link.stl"/>
         </geometry>
-        <material name="Blue">
-          <color rgba="0 0 255 1.0"/>
+        <material name="blue">
+          <color rgba="0 0 1 1"/>
         </material>
       </collision>
@@ -29,7 +29,5 @@
           <mesh filename="package://adept_s650_support/meshes/s650/visual/link_1.stl"/>
         </geometry>
-        <material name="Grey">
-          <color rgba="128 128 128 1.0"/>
-        </material>
+        <material name="adept_grey"/>
       </visual>
       <collision>
@@ -38,7 +36,5 @@
           <mesh filename="package://adept_s650_support/meshes/s650/collision/link_1.stl"/>
         </geometry>
-        <material name="Blue">
-          <color rgba="0 0 255 1.0"/>
-        </material>
+        <material name="blue"/>
       </collision>
     </link>
@@ -49,7 +45,5 @@
           <mesh filename="package://adept_s650_support/meshes/s650/visual/link_2.stl"/>
         </geometry>
-        <material name="Grey">
-          <color rgba="128 128 128 1.0"/>
-        </material>
+        <material name="adept_grey"/>
       </visual>
       <collision>
@@ -58,7 +52,5 @@
           <mesh filename="package://adept_s650_support/meshes/s650/collision/link_2.stl"/>
         </geometry>
-        <material name="Blue">
-          <color rgba="0 0 255 1.0"/>
-        </material>
+        <material name="blue"/>
       </collision>
     </link>
@@ -69,7 +61,5 @@
           <mesh filename="package://adept_s650_support/meshes/s650/visual/link_3.stl"/>
         </geometry>
-        <material name="Grey">
-          <color rgba="128 128 128 1.0"/>
-        </material>
+        <material name="adept_grey"/>
       </visual>
       <collision>
@@ -78,7 +68,5 @@
           <mesh filename="package://adept_s650_support/meshes/s650/collision/link_3.stl"/>
         </geometry>
-        <material name="Blue">
-          <color rgba="0 0 255 1.0"/>
-        </material>
+        <material name="blue"/>
       </collision>
     </link>
@@ -89,7 +77,5 @@
           <mesh filename="package://adept_s650_support/meshes/s650/visual/link_4.stl"/>
         </geometry>
-        <material name="Grey">
-          <color rgba="128 128 128 1.0"/>
-        </material>
+        <material name="adept_grey"/>
       </visual>
       <collision>
@@ -98,7 +84,5 @@
           <mesh filename="package://adept_s650_support/meshes/s650/collision/link_4.stl"/>
         </geometry>
-        <material name="Blue">
-          <color rgba="0 0 255 1.0"/>
-        </material>
+        <material name="blue"/>
       </collision>
     </link>
@@ -109,7 +93,5 @@
           <mesh filename="package://adept_s650_support/meshes/s650/visual/link_5.stl"/>
         </geometry>
-        <material name="Grey">
-          <color rgba="128 128 128 1.0"/>
-        </material>
+        <material name="adept_grey"/>
       </visual>
       <collision>
@@ -118,7 +100,5 @@
           <mesh filename="package://adept_s650_support/meshes/s650/collision/link_5.stl"/>
         </geometry>
-        <material name="Blue">
-          <color rgba="0 0 255 1.0"/>
-        </material>
+        <material name="blue"/>
       </collision>
     </link>
@@ -129,7 +109,5 @@
           <mesh filename="package://adept_s650_support/meshes/s650/visual/link_6.stl"/>
         </geometry>
-        <material name="Gray">
-          <color rgba="100 100 100 1.0"/>
-        </material>
+        <material name="adept_grey"/>
       </visual>
       <collision>
@@ -138,7 +116,5 @@
           <mesh filename="package://adept_s650_support/meshes/s650/collision/link_6.stl"/>
         </geometry>
-        <material name="Blue">
-          <color rgba="0 0 255 1.0"/>
-        </material>
+        <material name="blue"/>
       </collision>
     </link>
